Commit message: Create a maze model in gazebo

File: mousebot/urdf/mousebot.urdf (robot description, URDF)
Before this commit: robot mousebot, 6 links, 5 joints
Joints:
- joint hokuyo_joint: origin xyz=0 0 0.04 rpy=0 0 1.570796 -> xyz=0 0 0.03 rpy=0 0 1.570796

Commit message: comment out back two wheels

File: mousebot/urdf/mousebot.urdf (robot description, URDF)
Before this commit: robot mousebot, 6 links, 5 joints
Links:
- removed link BL_wheel
- removed link BR_wheel
Joints:
- removed joint BL_wheel_cont
- removed joint BR_wheel_cont

Commit message: Add new robot model

File: mousebot/urdf/mousebot.urdf (robot description, URDF)
Before this commit: robot mousebot, 4 links, 3 joints
Links:
- removed link FL_wheel
- removed link FR_wheel
- added link L_wheel, mass 0.010162; collision mesh filename=package://mousebot/meshes/L_wheel_col.STL; visual mesh filename=package://mousebot/meshes/L_wheel.STL
- added link R_wheel, mass 0.010162; collision mesh filename=package://mousebot/meshes/R_wheel_col.STL; visual mesh filename=package://mousebot/meshes/R_wheel.STL
- link mousebot: mass 0.0546391744414753 -> 0.0517193970626456
Joints:
- removed joint FL_wheel_cont
- removed joint FR_wheel_cont
- added joint L_wheel_cont: type continuous, parent mousebot, child L_wheel, origin xyz=-0.03556 0 0.0127 rpy=0 0 0, axis -1 0 0, limit effort=0 velocity=200
- added joint R_wheel_cont: type continuous, parent mousebot, child R_wheel, origin xyz=0.03556 0 0.0127 rpy=0 0 0, axis -1 0 0, limit effort=0 velocity=200

Commit message: Shrink Mousebot and fix axis orientation

File: mousebot/urdf/mousebot.urdf (robot description, URDF)
Before this commit: robot mousebot, 4 links, 3 joints
Links:
- link L_wheel: mass 0.010162 -> 0.010055
- link R_wheel: mass 0.010162 -> 0.010055
- link mousebot: mass 0.0517193970626456 -> 0.147
Joints:
- joint L_wheel_cont: axis -1 0 0 -> 0 1 0; origin xyz=-0.03556 0 0.0127 rpy=0 0 0 -> xyz=0 0.03175 0.0127 rpy=0 0 0
- joint R_wheel_cont: axis -1 0 0 -> 0 1 0; origin xyz=0.03556 0 0.0127 rpy=0 0 0 -> xyz=0 -0.03175 0.0127 rpy=0 0 0

Commit message: Fix bugs with LIDAR

File: mousebot/urdf/mousebot.urdf (robot description, URDF)
Before this commit: robot mousebot, 4 links, 3 joints
Joints:
- joint hokuyo_joint: origin xyz=0 0 0.03 rpy=0 0 1.570796 -> xyz=0 0 0.03 rpy=0 0 3.1415926
